File: esp_weather_pcb/esp_weather_pcb.kicad_pcb (KiCad board)
At the start: 2 copper layers, 65 x 75 mm, 6 parts, among them U1 esp32_38P_Left, U2 esp32_38P_Right

Commit message: updated pcb
Parts:
- added Pads_Right1: esp32_38P_Right_Pads, esp32_devboards:esp32_38P_right_pads, F.Cu at (99.9, 86.0)
- added Pads_left1: esp32_38P_Left_Pads, esp32_devboards:esp32_38P_left_Pads, F.Cu at (65.0, 86.0)
- added REF**: MountingHole_2.2mm_M2, MountingHole:MountingHole_2.2mm_M2, F.Cu at (107.0, 112.0)
- added REF**: MountingHole_2.2mm_M2, MountingHole:MountingHole_2.2mm_M2, F.Cu at (58.0, 53.0)
- added REF**: MountingHole_2.2mm_M2, MountingHole:MountingHole_2.2mm_M2, F.Cu at (107.0, 53.0)
- added REF**: MountingHole_2.2mm_M2, MountingHole:MountingHole_2.2mm_M2, F.Cu at (58.0, 112.0)
- moved Disp1 28.0 mm to (104.0, 88.0), turned to 90 degrees
- moved Outside1 9.06 mm to (61.0, 106.0), turned to -90 degrees
- moved Temp1 5.10 mm to (104.0, 103.0), turned to 90 degrees
- renumbered U1 to ESP_Left1, U2 to ESP_Right1
Connections:
- net Net-(Outside1-D) renamed P16
- ESP_Left1 pad 10: unconnected-(U1-P26-Pad10) -> Net-(ESP_Left1-P26)
- ESP_Left1 pad 11: unconnected-(U1-P27-Pad11) -> Net-(ESP_Left1-P27)
- ESP_Left1 pad 12: unconnected-(U1-P14-Pad12) -> Net-(ESP_Left1-P14)
- ESP_Left1 pad 13: unconnected-(U1-P12-Pad13) -> Net-(ESP_Left1-P12)
- ESP_Left1 pad 15: unconnected-(U1-P13-Pad15) -> Net-(ESP_Left1-P13)
- ESP_Left1 pad 16: unconnected-(U1-FLASH_D2-Pad16) -> Net-(ESP_Left1-FLASH_D2)
- ESP_Left1 pad 17: unconnected-(U1-FLASH_D3-Pad17) -> Net-(ESP_Left1-FLASH_D3)
- ESP_Left1 pad 18: unconnected-(U1-FLASH_CMD-Pad18) -> Net-(ESP_Left1-FLASH_CMD)
- ESP_Left1 pad 19: unconnected-(U1-5V-Pad19) -> Net-(ESP_Left1-5V)
- ESP_Left1 pad 2: unconnected-(U1-EN-Pad2) -> Net-(ESP_Left1-EN)
- ESP_Left1 pad 3: unconnected-(U1-P36-Pad3) -> Net-(ESP_Left1-P36)
- ESP_Left1 pad 4: unconnected-(U1-P39-Pad4) -> Net-(ESP_Left1-P39)
- ESP_Left1 pad 5: unconnected-(U1-P34-Pad5) -> Net-(ESP_Left1-P34)
- ESP_Left1 pad 6: unconnected-(U1-P35-Pad6) -> Net-(ESP_Left1-P35)
- ESP_Left1 pad 7: unconnected-(U1-P32-Pad7) -> Net-(ESP_Left1-P32)
- ESP_Left1 pad 8: unconnected-(U1-P33-Pad8) -> Net-(ESP_Left1-P33)
- ESP_Left1 pad 9: unconnected-(U1-P25-Pad9) -> Net-(ESP_Left1-P25)
- ESP_Right1 pad 20: unconnected-(U2-FLASH_CLK-Pad20) -> Net-(ESP_Right1-FLASH_CLK)
- ESP_Right1 pad 21: unconnected-(U2-FLASH_D0-Pad21) -> Net-(ESP_Right1-FLASH_D0)
- ESP_Right1 pad 22: unconnected-(U2-FLASH_D1-Pad22) -> Net-(ESP_Right1-FLASH_D1)
- ESP_Right1 pad 23: unconnected-(U2-P15-Pad23) -> Net-(ESP_Right1-P15)
- ESP_Right1 pad 24: unconnected-(U2-P2-Pad24) -> Net-(ESP_Right1-P2)
- ESP_Right1 pad 25: unconnected-(U2-P0-Pad25) -> Net-(ESP_Right1-P0)
- ESP_Right1 pad 26: unconnected-(U2-P4-Pad26) -> Net-(ESP_Right1-P4)
- ESP_Right1 pad 28: unconnected-(U2-P17-Pad28) -> Net-(ESP_Right1-P17)
- ESP_Right1 pad 29: unconnected-(U2-P5-Pad29) -> Net-(ESP_Right1-P5)
- ESP_Right1 pad 30: unconnected-(U2-P18-Pad30) -> Net-(ESP_Right1-P18)
- ESP_Right1 pad 31: unconnected-(U2-P19-Pad31) -> Net-(ESP_Right1-P19)
- ESP_Right1 pad 34: unconnected-(U2-RX-Pad34) -> Net-(ESP_Right1-RX)
- ESP_Right1 pad 35: unconnected-(U2-TX-Pad35) -> Net-(ESP_Right1-TX)
- ESP_Right1 pad 37: unconnected-(U2-P23-Pad37) -> Net-(ESP_Right1-P23)
Routing:
- net 3V3: track 124.9 -> 141.6 mm
- net SCL: track 67.3 -> 58.3 mm
- net P16: track 43.8 -> 52.0 mm
- net Net-(ESP_Right1-TX): track 0.00 -> 6.00 mm
- net Net-(ESP_Right1-RX): track 0.00 -> 6.00 mm
- net Net-(ESP_Right1-P5): track 0.00 -> 6.00 mm
- net Net-(ESP_Right1-P4): track 0.00 -> 6.00 mm
- net Net-(ESP_Right1-P23): track 0.00 -> 6.00 mm
- net Net-(ESP_Right1-P2): track 0.00 -> 6.00 mm
- net Net-(ESP_Right1-P19): track 0.00 -> 6.00 mm
- net Net-(ESP_Right1-P18): track 0.00 -> 6.00 mm
- net Net-(ESP_Right1-P17): track 0.00 -> 6.00 mm
- net Net-(ESP_Right1-P15): track 0.00 -> 6.00 mm
- net Net-(ESP_Right1-P0): track 0.00 -> 6.00 mm
- net Net-(ESP_Right1-FLASH_D1): track 0.00 -> 6.00 mm
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Other:
- board size 65 x 75 mm -> 55 x 65 mm
